File: Connectors.kicad_sch (KiCad schematic)
At the start: 16 parts, among them J16 USB_A_Stacked, J23 HR911130A, J24 HR911130A, U1 TPS2065CDBV

Commit message: Restructured v0.1 for easier worktree use
Changed lines of the file:
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@@
 	(title_block
 		(title "OpenMower SABO Mainboard for Series I & II")
-		(date "2025-05-22")
-		(rev "v0.2")
+		(date "2025-02-26")
+		(rev "v0.1")
 		(company "Apeheanger <joerg@ebeling.ws> for OpenMower")
 		(comment 1 "This design is licensed under CC BY-NC 4.0")
@@
 	(wire
 		(pts
+			(xy 109.22 173.99) (xy 109.22 168.91)
+		)
+		(stroke
+			(width 0)
+			(type default)
+		)
+	)
+	(wire
+		(pts
 			(xy 73.66 205.74) (xy 76.2 205.74)
 		)
@@
 			)
 		)
-		(property "MPN" ""
-			(at 254 137.16 0)
-			(effects
-				(font
-					(size 1.27 1.27)
-				)
-			)
-		)
 		(pin "4"
 		)
@@
 			)
 		)
-		(property "MPN" ""
-			(at 64.77 152.4 0)
-			(effects
-				(font
-					(size 1.27 1.27)
-				)
-			)
-		)
 		(pin "2"
 		)
@@
 			)
 		)
-		(property "MPN" ""
-			(at 105.41 160.02 0)
-			(effects
-				(font
-					(size 1.27 1.27)
-				)
-			)
-		)
 		(pin "1"
 		)
@@
 			)
 		)
-		(property "MPN" ""
-			(at 105.41 147.32 0)
-			(effects
-				(font
-					(size 1.27 1.27)
-				)
-			)
-		)
 		(pin "1"
 		)
@@
 		(dnp no)
 		(property "Reference" "C5"
-			(at 105.41 165.354 90)
+			(at 105.41 166.37 90)
 			(effects
 				(font
@@
 		)
 		(property "Value" "100nF@50V"
-			(at 112.522 171.704 90)
+			(at 105.41 168.91 90)
 			(effects
 				(font
@@
 			)
 		)
-		(property "MPN" ""
-			(at 105.41 168.91 0)
-			(effects
-				(font
-					(size 1.27 1.27)
-				)
-			)
-		)
 		(pin "2"
 		)
@@
 			)
 		)
-		(property "MPN" ""
-			(at 82.55 149.86 0)
-			(effects
-				(font
-					(size 1.27 1.27)
-				)
-			)
-		)
 		(pin "5"
 		)
@@
 			)
 		)
-		(property "MPN" ""
-			(at 63.5 147.32 0)
-			(effects
-				(font
-					(size 1.27 1.27)
-				)
-			)
-		)
 		(pin "2"
 		)
@@
 			)
 		)
-		(property "MPN" ""
-			(at 227.33 240.03 0)
-			(effects
-				(font
-					(size 1.27 1.27)
-				)
-			)
-		)
 		(pin "2"
 		)
@@
 			)
 		)
-		(property "MPN" ""
-			(at 227.33 139.7 0)
-			(effects
-				(font
-					(size 1.27 1.27)
-				)
-			)
-		)
 		(pin "2"
 		)
@@
 			)
 		)
-		(property "MPN" ""
-			(at 73.66 190.5 0)
-			(effects
-				(font
-					(size 1.27 1.27)
-				)
-			)
-		)
 		(pin "3"
 		)
@@
 			)
 		)
-		(property "MPN" ""
-			(at 231.14 199.39 0)
-			(effects
-				(font
-					(size 1.27 1.27)
-				)
-			)
-		)
 		(pin "2"
 		)
@@
 			)
 		)
-		(property "MPN" ""
-			(at 82.55 135.89 0)
-			(effects
-				(font
-					(size 1.27 1.27)
-				)
-			)
-		)
 		(pin "2"
 		)
@@
 			)
 		)
-		(property "MPN" ""
-			(at 231.14 111.76 0)
-			(effects
-				(font
-					(size 1.27 1.27)
-				)
-			)
-		)
 		(pin "2"
 		)
@@
 			)
 		)
-		(property "MPN" ""
-			(at 227.33 152.4 0)
-			(effects
-				(font
-					(size 1.27 1.27)
-				)
-			)
-		)
 		(pin "2"
 		)
@@
 	(symbol
 		(lib_id "power:GND")
-		(at 109.22 168.91 90)
+		(at 109.22 173.99 90)
 		(mirror x)
 		(unit 1)
@@
 		(fields_autoplaced yes)
 		(property "Reference" "#PWR016"
-			(at 115.57 168.91 0)
+			(at 115.57 173.99 0)
 			(effects
 				(font
@@
 		)
 		(property "Value" "GND"
-			(at 113.03 168.9099 90)
+			(at 113.03 173.9899 90)
 			(effects
 				(font
@@
 		)
 		(property "Footprint" ""
-			(at 109.22 168.91 0)
+			(at 109.22 173.99 0)
 			(effects
 				(font
@@
 		)
 		(property "Datasheet" ""
-			(at 109.22 168.91 0)
+			(at 109.22 173.99 0)
 			(effects
 				(font
@@
 		)
 		(property "Description" "Power symbol creates a global label with name \"GND\" , ground"
-			(at 109.22 168.91 0)
+			(at 109.22 173.99 0)
 			(effects
 				(font
@@
 			)
 		)
-		(property "MPN" ""
-			(at 227.33 227.33 0)
-			(effects
-				(font
-					(size 1.27 1.27)
-				)
-			)
-		)
 		(pin "2"
 		)
@@
 			)
 		)
-		(property "MPN" ""
-			(at 254 224.79 0)
-			(effects
-				(font
-					(size 1.27 1.27)
-				)
-			)
-		)
