File: Connectors.kicad_sch (KiCad schematic)
At the start: 12 parts, among them J16 USB_A_Stacked, J24 HR911130A, U1 TPS2065CDBVR

Commit message: KiCAD 10.x, Mow-ESC-Fuse, Improve power traces
Parts:
- J24: MANUFACTURER HanRun -> (none); Manufacturer (none) -> HanRun; PACKAGE (none) -> None; Package None -> (none)
