File: DCDC.kicad_sch (KiCad schematic)
At the start: 25 parts, among them U5 LM76005RNPR

Commit message: BOM optimization
Other:
- title: OpenMower SABO Mainboard for Series I & II -> OpenMower SABO Carrierboard for Series I & II
Changed lines of the file:
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@@
 	(paper "A3")
 	(title_block
-		(title "OpenMower SABO Mainboard for Series I & II")
-		(date "2025-10-05")
-		(rev "v0.3")
+		(title "OpenMower SABO Carrierboard for Series I & II")
+		(date "2025-10-12")
+		(rev "v0.4")
 		(company "Apeheanger <joerg@ebeling.ws> for OpenMower")
 		(comment 1 "This design is licensed under CC BY-NC 4.0")
@@
 			)
 		)
-		(property "Description" "Unpolarized capacitor"
+		(property "Description" "50V 100nF X7R ±10% 0402 Multilayer Ceramic Capacitors MLCC"
 			(at 325.12 119.38 0)
 			(effects
@@
 			)
 		)
-		(property "Description" "Unpolarized capacitor"
+		(property "Description" "50V 100nF X7R ±10% 0402 Multilayer Ceramic Capacitors MLCC"
 			(at 313.69 119.38 0)
 			(effects
