File: RobotConnectorsSeries2.kicad_sch (KiCad schematic)
At the start: 15 parts, among them U6 LM339

Commit message: Update Status & BOM
Parts:
- S2-J2: now fitted; now in the parts list
- S2-J7: footprint local_Connectors:Molex_Milli-Grid_878311420 -> local_Connectors:Molex_Milli-Grid_878311419; MFPN 878312619 -> 878311419
- S2-J8: MFPN 878311019 -> 878311041; now fitted; now in the parts list
Changed lines of the file:
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@@
 			)
 		)
-		(property "Footprint" "local_Connectors:Molex_Milli-Grid_878311420"
+		(property "Footprint" "local_Connectors:Molex_Milli-Grid_878311419"
 			(at 209.55 106.68 0)
 			(effects
@@
 			)
 		)
-		(property "MFPN" "878312619"
+		(property "MFPN" "878311419"
 			(at 209.55 106.68 0)
 			(effects
@@
 		(unit 1)
 		(exclude_from_sim no)
-		(in_bom no)
-		(on_board yes)
-		(dnp yes)
+		(in_bom yes)
+		(on_board yes)
+		(dnp no)
 		(property "Reference" "S2-J8"
 			(at 265.43 142.494 0)
@@
 			)
 		)
-		(property "MFPN" "878311019"
+		(property "MFPN" "878311041"
 			(at 264.16 153.67 0)
 			(effects
@@
 		(unit 1)
 		(exclude_from_sim no)
-		(in_bom no)
-		(on_board yes)
-		(dnp yes)
+		(in_bom yes)
+		(on_board yes)
+		(dnp no)
 		(property "Reference" "S2-J2"
 			(at 199.39 20.066 0)

Commit message: Update status
Other:
- note added: "----------- DESIGN FAULTS ---------- 1. Hall Sensors SAU12996 and SAU13124 will not work reliable with R_{Sense} = 330. R9, R10 & R28 need to be changed to 120 Ohm. 2. In consequence of 1. R23 need to be changed to 3k3 to get a V_{Ref} of 1.24V 3. Comparator V_{Ref} inputs Pin 4, 6 & 8 need an 100k R in series so that an oscillation comparator doesn't affect V_{Ref}. 4. The unused "C" comparator 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"
- note added: "Top-Stop Hall = SAU13124, 1503 (3-pin) Vcc | LowSide-R | Idle | Active | ---------------------------------- 5V | 120 | 1.73V | 0.73V |"
- note added: "Wheel-Lift Hall = SAU12996, 1308 (2-pin) ======================================== Vcc | LowSide-R | Idle | Active | ---------------------------------- 5V | 120 | 1.85V | 0.74V |"
- note removed: "SAU??? (2-pin) SAU13124, 1503 (3-pin) ====================== Vcc | LowSide-R | Idle | Active | --------------------------------- 5V | 220 | Not working | 5V | 330 | 3.3V | 2V | 5V | 470 | 3.4V | 2.8 | 5V | 1000 | Not working |"
- moved on the sheet: C87, R10, R28, R9, S2-J10, S2-J2, S2-J7, U6A, U6B, U6D

Commit message: Prepare v0.2
Parts:
- removed R9: 330, Resistor_SMD:R_0603_1608Metric, symbol Device:R
- added Q3: AO3401A, Package_TO_SOT_SMD:SOT-23, symbol Transistor_FET:AO3401A
- added R39, R40, R41, R42, R89: 10k, Resistor_SMD:R_0603_1608Metric_Pad0.98x0.95mm_HandSolder, symbol Device:R
- added R43, R90: 3k3, Resistor_SMD:R_0603_1608Metric_Pad0.98x0.95mm_HandSolder, symbol Device:R
- added R91: 10k, Resistor_SMD:R_0402_1005Metric, symbol Device:R
- R10, R28: value 330 -> 120; footprint Resistor_SMD:R_0603_1608Metric -> Resistor_SMD:R_0603_1608Metric_Pad0.98x0.95mm_HandSolder; JLC C23138 -> C22787
- R23: value 11k -> 3k3; footprint Resistor_SMD:R_0402_1005Metric -> Resistor_SMD:R_0603_1608Metric_Pad0.98x0.95mm_HandSolder; JLC C25749 -> C22978
- R27: value 10k -> 120; footprint Resistor_SMD:R_0402_1005Metric -> Resistor_SMD:R_0603_1608Metric_Pad0.98x0.95mm_HandSolder; JLC C25744 -> C22787
- S2-J1: footprint local_Connectors:Molex_Mini-Fit_Jr_5566-16A_2x08_P4.20mm_Vertical -> local_Connectors:CONN-TH_X9357WV-2X08HN-N2SN; Alternative (none) -> XKB Connection X9357WV-2x08HN-N2SN. ATTENTION: Different Fo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; JLC C5339222 -> C388779
- S2-J7: footprint local_Connectors:Molex_Milli-Grid_878311419 -> local_Connectors:Molex_Milli-Grid_878311420
Connections:
- net 5V: now also Q3.3 (D), R91.2; no longer C53.1, C87.1, R27.1, S2-J7.3 (Pin_3), U6.3 (V+)
- net GND: now also R27.2, R40.2, R43.2, R90.2; no longer S2-J2.5 (Pin_5)
- net at S2-J7.2 (Pin_2), U6.9 (+): now also R27.1
- net at U6.10 (-): now also R39.2
- net at U6.11 (+): now also R40.1
- removed net 2.6V_REF: R23.1, R27.2, U6.4 (-), U6.6 (-), U6.8 (-)
- net BTN_~{CE} renamed BTN_~{CE}_5V
- net LATCH_LOAD renamed LATCH_LOAD_5V
- net LCD_IN_X renamed LCD_IN_X_5V
- net LCD_IN_Y renamed LCD_IN_Y_5V
- net LCD_IN_Z renamed LCD_IN_Z_5V
- net OE renamed OE_5V
- net SPI_CLK renamed SPI_CLK_5V
- net SPI_RX renamed SPI_RX_5V
- net SPI_TX renamed SPI_TX_5V
- new net 1.24V_REF_A: R42.2, R43.1, U6.4 (-)
- new net 1.24V_REF_B: R89.2, R90.1, U6.6 (-)
- new net 1.24V_REF_D: R23.1, R41.2, U6.8 (-)
- new net 5V_HALL: C53.1, C87.1, Q3.2 (S), R39.1, R41.1, R42.1, R89.1, S2-J7.3 (Pin_3), U6.3 (V+)
- new net HALL_~{EN}_5V: Q3.1 (G), R91.1
- new net UI_~{CON}: S2-J2.5 (Pin_5)
- no-connect marks 27 -> 25
Other:
- note removed: "----------- DESIGN FAULTS ---------- 1. Hall Sensors SAU12996 and SAU13124 will not work reliable with R_{Sense} = 330. R9, R10 & R28 need to be changed to 120 Ohm. 2. In consequence of 1. R23 need to be changed to 3k3 to get a V_{Ref} of 1.24V 3. Comparator V_{Ref} inputs Pin 4, 6 & 8 need an 100k R in series so that an oscillation comparator doesn't affect V_{Ref}. 4. The unused "C" comparator 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"
- moved on the sheet: R23, U6C, U6D

Commit message: Add RoHS Compliance Summary
Parts:
- U6: JLC C7948 -> (none); LCSC Part # (none) -> C7948

Commit message: Add Series-II emergency backup plan
Parts:
- added J11, J12, J13: Conn_01x03_Male, Connector_JST:JST_XH_B3B-XH-A_1x03_P2.50mm_Vertical, symbol Connector:Conn_01x03_Male
- S2-J8: now not fitted; now left out of the parts list
Connections:
- net 5V: now also J11.1 (Pin_1), J12.1 (Pin_1), J13.1 (Pin_1)
- net GND: now also J11.3 (Pin_3), J12.3 (Pin_3), J13.3 (Pin_3)
- net HALL0_5V: now also J11.2 (Pin_2)
- net HALL1_5V: now also J12.2 (Pin_2)
- net HALL2_5V: now also J13.2 (Pin_2)
Other:
- note added: "Backup plan"

Commit message: Finish v0.2 schematic and ERC
Connections:
- net LCD_MOSI_3V: now reaches S2-J2.21 (Pin_21)
- net LCD_VCC_3V: now reaches S2-J2.22 (Pin_22)
- net LCD_IN_MISC1_3V: now reaches S2-J2.24 (Pin_24)
- net LCD_IN_X_5V renamed LCD_IN_MISC2_3V
- net LCD_IN_Y_5V renamed LCD_CLK_3V
- net LCD_IN_Z_5V renamed LCD_~{CE}_3V
- no-connect marks 25 -> 22
Other:
- note added: "(always high during RE)"
- note added: "LCD_IN_MISC2: 1-3 low-strobes @ end of ~{CE} phase during RE"
Changed lines of the file:
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@@
 	(title_block
 		(title "OpenMower SABO Mainboard for Series I & II")
-		(date "2025-05-04")
+		(date "2025-05-22")
 		(rev "v0.2")
 		(company "Apeheanger <joerg@ebeling.ws> for OpenMower")
@@
 		)
 	)
+	(text "(always high during RE)"
+		(exclude_from_sim no)
+		(at 221.234 67.31 0)
+		(effects
+			(font
+				(size 1.27 1.27)
+			)
+		)
+	)
 	(text "Front-Left-Lift"
 		(exclude_from_sim no)
@@
 		(exclude_from_sim no)
 		(at 86.868 85.598 0)
+		(effects
+			(font
+				(size 1.27 1.27)
+			)
+		)
+	)
+	(text "LCD_IN_MISC2:\n1-3 low-strobes\n@ end of ~{CE} phase\nduring RE"
+		(exclude_from_sim no)
+		(at 152.4 56.134 0)
 		(effects
 			(font
@@
 	)
 	(no_connect
-		(at 204.47 62.23)
-	)
-	(no_connect
 		(at 229.87 115.57)
 	)
@@
 	)
 	(no_connect
-		(at 191.77 62.23)
-	)
-	(no_connect
 		(at 217.17 120.65)
 	)
@@
 	(no_connect
 		(at 271.78 148.59)
-	)
-	(no_connect
-		(at 204.47 64.77)
 	)
 	(no_connect
@@
 	(wire
 		(pts
+			(xy 180.34 62.23) (xy 191.77 62.23)
+		)
+		(stroke
+			(width 0)
+			(type default)
+		)
+	)
+	(wire
+		(pts
 			(xy 229.87 107.95) (xy 237.49 107.95)
 		)
@@
 		)
 	)
+	(wire
+		(pts
+			(xy 204.47 62.23) (xy 209.55 62.23)
+		)
+		(stroke
+			(width 0)
+			(type default)
+		)
+	)
 	(bus
 		(pts
@@
 		(pts
 			(xy 83.82 185.42) (xy 86.36 185.42)
+		)
+		(stroke
+			(width 0)
+			(type default)
+		)
+	)
+	(wire
+		(pts
+			(xy 204.47 64.77) (xy 209.55 64.77)
 		)
 		(stroke
@@
 		)
 	)
+	(hierarchical_label "LCD_IN_MISC2_3V"
+		(shape input)
+		(at 180.34 54.61 180)
+		(effects
+			(font
+				(size 1.27 1.27)
+			)
+			(justify right)
+		)
+	)
 	(hierarchical_label "BMC_YW"
 		(shape bidirectional)
@@
 		)
 	)
+	(hierarchical_label "LCD_VCC_3V"
+		(shape input)
+		(at 209.55 62.23 0)
+		(effects
+			(font
+				(size 1.27 1.27)
+			)
+			(justify left)
+		)
+	)
 	(hierarchical_label "LATCH_LOAD_5V"
 		(shape input)
@@
 		)
 	)
+	(hierarchical_label "LCD_CLK_3V"
+		(shape input)
+		(at 180.34 57.15 180)
+		(effects
+			(font
+				(size 1.27 1.27)
+			)
+			(justify right)
+		)
+	)
 	(hierarchical_label "HALL_~{EN}_5V"
 		(shape input)
@@
 		)
 	)
+	(hierarchical_label "LCD_MOSI_3V"
+		(shape input)
+		(at 180.34 62.23 180)
+		(effects
+			(font
+				(size 1.27 1.27)
+			)
+			(justify right)
+		)
+	)
 	(hierarchical_label "HALL2_5V"
 		(shape output)
@@
 		)
 	)
-	(hierarchical_label "LCD_IN_Y_5V"
-		(shape input)
-		(at 180.34 57.15 180)
-		(effects
-			(font
-				(size 1.27 1.27)
-			)
-			(justify right)
-		)
-	)
 	(hierarchical_label "OE_5V"
 		(shape input)
@@
 		)
 	)
+	(hierarchical_label "LCD_~{CE}_3V"
+		(shape input)
+		(at 209.55 59.69 0)
+		(effects
+			(font
+				(size 1.27 1.27)
+			)
+			(justify left)
+		)
+	)
 	(hierarchical_label "HALL0_5V"
 		(shape output)
@@
 		)
 	)
+	(hierarchical_label "LCD_IN_MISC1_3V"
+		(shape input)
+		(at 209.55 64.77 0)
+		(effects
+			(font
+				(size 1.27 1.27)
+			)
+			(justify left)
+		)
+	)
 	(hierarchical_label "LCD_BACKLIGHT_KATHODE"
 		(shape input)
@@
 		)
 	)
-	(hierarchical_label "LCD_IN_X_5V"
-		(shape input)
-		(at 180.34 54.61 180)
-		(effects
-			(font
-				(size 1.27 1.27)
-			)
-			(justify right)
-		)
-	)
-	(hierarchical_label "LCD_IN_Z_5V"
-		(shape input)
-		(at 209.55 59.69 0)
-		(effects
-			(font
-				(size 1.27 1.27)
-			)
-			(justify left)
-		)
-	)

Commit message: Finish v0.2 PCB and DRC
Parts:
- S2-J1: footprint local_Connectors:CONN-TH_X9357WV-2X08HN-N2SN -> local_Connectors:Molex_Mini-Fit_Jr_5566-16A_2x08_P4.20mm_Vertical; Alternative XKB Connection X9357WV-2x08HN-N2SN. ATTENTION: Different Fo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 -> (none); JLC C388779 -> C5339222
- S2-J2: DNP Y -> (none)
- S2-J5, S2-J6: FT Rotation Offset 180 -> 0; JLC C505075 -> (none); LCSC Part # (none) -> C400369; MF Molex -> (none); Manufacturer (none) -> Molex
- S2-J7: LCSC Part # (none) -> C17218801
Changed lines of the file:
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@@
 			)
 		)
-		(property "JLC" ""
-			(at 168.91 179.07 0)
-			(effects
-				(font
-					(size 1.27 1.27)
-				)
-				(hide yes)
-			)
-		)
 		(property "MPN" ""
 			(at 168.91 179.07 0)
@@
 			)
 		)
-		(property "MPN" ""
+		(property "LCSC Part #" "C17218801"
 			(at 222.25 115.57 0)
 			(effects
@@
 					(size 1.27 1.27)
 				)
+				(hide yes)
 			)
 		)
@@
 			)
 		)
-		(property "JLC" ""
-			(at 260.35 110.49 0)
-			(effects
-				(font
-					(size 1.27 1.27)
-				)
-				(hide yes)
-			)
-		)
 		(property "MPN" ""
 			(at 260.35 110.49 0)
@@
 			)
 		)
-		(property "JLC" ""
-			(at 250.19 44.45 0)
-			(effects
-				(font
-					(size 1.27 1.27)
-				)
-				(hide yes)
-			)
-		)
 		(property "MPN" ""
 			(at 250.19 44.45 0)
@@
 			)
 		)
-		(property "Description" "Generic connectable mounting pin connector, double row, 02x04, top/bottom pin numbering scheme (row 1: 1...pins_per_row, row2: pins_per_row+1 ... num_pins), script generated (kicad-library-utils/schlib/autogen/connector/)"
+		(property "Description" "2x4P 8P Micro-Fit(MX 3.0) Tin 3mm 4 -40℃~+105℃ 8.5A 2 3mm Brass Standing paste SMD,P=3mm Wire To Board Connector ROHS"
 			(at 77.47 120.65 0)
 			(effects
@@
 			)
 		)
-		(property "MF" "Molex"
+		(property "Manufacturer" "Molex"
 			(at 77.47 120.65 0)
 			(effects
@@
 			)
 		)
-		(property "JLC" "C505075"
+		(property "LCSC Part #" "C400369"
 			(at 77.47 120.65 0)
 			(effects
@@
 			)
 		)
-		(property "FT Rotation Offset" "180"
+		(property "FT Rotation Offset" "0"
 			(at 77.47 120.65 0)
 			(effects
@@
 			)
 		)
-		(property "MPN" ""
-			(at 77.47 120.65 0)
-			(effects
-				(font
-					(size 1.27 1.27)
-				)
-			)
-		)
 		(pin "1"
 		)
@@
 			)
 		)
-		(property "DNP" "Y"
-			(at 196.85 52.07 0)
-			(effects
-				(font
-					(size 1.27 1.27)
-				)
-				(hide yes)
-			)
-		)
-		(property "MPN" ""
-			(at 196.85 52.07 0)
-			(effects
-				(font
-					(size 1.27 1.27)
-				)
-			)
-		)
 		(pin "4"
 		)
@@
 			)
 		)
-		(property "JLC" ""
-			(at 138.43 180.34 0)
-			(effects
-				(font
-					(size 1.27 1.27)
-				)
-				(hide yes)
-			)
-		)
 		(property "MPN" ""
 			(at 138.43 180.34 0)
@@
 			)
 		)
-		(property "JLC" ""
-			(at 190.5 110.49 0)
-			(effects
-				(font
-					(size 1.27 1.27)
-				)
-				(hide yes)
-			)
-		)
 		(property "MPN" ""
 			(at 190.5 110.49 0)
@@
 			)
 		)
-		(property "Footprint" "local_Connectors:CONN-TH_X9357WV-2X08HN-N2SN"
+		(property "Footprint" "local_Connectors:Molex_Mini-Fit_Jr_5566-16A_2x08_P4.20mm_Vertical"
 			(at 77.47 40.64 0)
 			(effects
@@
 			)
 		)
-		(property "Alternative" "XKB Connection X9357WV-2x08HN-N2SN. ATTENTION: Different Footprint"
+		(property "JLC" "C5339222"
 			(at 77.47 40.64 0)
 			(effects
@@
 			)
 		)
-		(property "JLC" "C388779"
-			(at 77.47 40.64 0)
-			(effects
-				(font
-					(size 1.27 1.27)
-				)
-				(hide yes)
-			)
-		)
-		(property "MPN" ""
-			(at 77.47 40.64 0)
-			(effects
-				(font
-					(size 1.27 1.27)
-				)
-			)
-		)
 		(pin "1"
 		)
@@
 			)
 		)
-		(property "Description" "Generic connectable mounting pin connector, double row, 02x04, top/bottom pin numbering scheme (row 1: 1...pins_per_row, row2: pins_per_row+1 ... num_pins), script generated (kicad-library-utils/schlib/autogen/connector/)"
+		(property "Description" "2x4P 8P Micro-Fit(MX 3.0) Tin 3mm 4 -40℃~+105℃ 8.5A 2 3mm Brass Standing paste SMD,P=3mm Wire To Board Connector ROHS"
 			(at 77.47 81.28 0)
 			(effects
@@
 			)
 		)
-		(property "MF" "Molex"
+		(property "Manufacturer" "Molex"
 			(at 77.47 81.28 0)
 			(effects
@@
 			)
 		)
-		(property "JLC" "C505075"
+		(property "LCSC Part #" "C400369"
 			(at 77.47 81.28 0)
 			(effects
@@
 			)
 		)
-		(property "FT Rotation Offset" "180"
+		(property "FT Rotation Offset" "0"
 			(at 77.47 81.28 0)
 			(effects
@@
 			)
 		)
-		(property "MPN" ""
-			(at 77.47 81.28 0)
-			(effects
-				(font
-					(size 1.27 1.27)
-				)
-			)
-		)

Commit message: Additional Infos
Changed lines of the file:
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@@
 					(size 1.27 1.27)
 				)
+				(hide yes)
 			)
 		)
