File: RobotConnectorsSeries2.kicad_sch (KiCad schematic)
At the start: 21 parts, among them U49 LM2903DR, U50 LM2903DR

Commit message: Production state
Parts:
- S2-J5, S2-J6: value Conn_02x04_Top_Bottom -> Conn_02x04_Top_Bottom_MountingPin
Changed lines of the file:
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@@
 	(title_block
 		(title "OpenMower SABO Carrierboard for Series I & II")
-		(date "2025-10-12")
+		(date "2026-04-04")
 		(rev "v0.4")
 		(company "Apeheanger <joerg@ebeling.ws> for OpenMower")
@@
 		)
 		(instances
-			(project ""
+			(project "hw-openmower-sabo"
 				(path "/e12e8a63-1d1b-4736-9aba-a87a258b2b11/7a7dfcf0-39e0-4eb7-9f4b-f66d7afbe41f/dd64c4b9-f40c-48f2-9722-a05c0658867e"
 					(reference "U49")
@@
 		)
 		(instances
-			(project ""
+			(project "hw-openmower-sabo"
 				(path "/e12e8a63-1d1b-4736-9aba-a87a258b2b11/7a7dfcf0-39e0-4eb7-9f4b-f66d7afbe41f/dd64c4b9-f40c-48f2-9722-a05c0658867e"
 					(reference "U49")
@@
 		)
 		(instances
-			(project ""
+			(project "hw-openmower-sabo"
 				(path "/e12e8a63-1d1b-4736-9aba-a87a258b2b11/7a7dfcf0-39e0-4eb7-9f4b-f66d7afbe41f/dd64c4b9-f40c-48f2-9722-a05c0658867e"
 					(reference "U50")
@@
 		)
 		(instances
-			(project ""
+			(project "hw-openmower-sabo"
 				(path "/e12e8a63-1d1b-4736-9aba-a87a258b2b11/7a7dfcf0-39e0-4eb7-9f4b-f66d7afbe41f/dd64c4b9-f40c-48f2-9722-a05c0658867e"
 					(reference "U50")
@@
 			)
 		)
-		(property "Value" "Conn_02x04_Top_Bottom"
+		(property "Value" "Conn_02x04_Top_Bottom_MountingPin"
 			(at 78.74 111.76 0)
 			(effects
@@
 		)
 		(instances
-			(project ""
+			(project "hw-openmower-sabo"
 				(path "/e12e8a63-1d1b-4736-9aba-a87a258b2b11/7a7dfcf0-39e0-4eb7-9f4b-f66d7afbe41f/dd64c4b9-f40c-48f2-9722-a05c0658867e"
 					(reference "U49")
@@
 		)
 		(instances
-			(project ""
+			(project "hw-openmower-sabo"
 				(path "/e12e8a63-1d1b-4736-9aba-a87a258b2b11/7a7dfcf0-39e0-4eb7-9f4b-f66d7afbe41f/dd64c4b9-f40c-48f2-9722-a05c0658867e"
 					(reference "U50")
@@
 		)
 		(instances
-			(project ""
+			(project "hw-openmower-sabo"
 				(path "/e12e8a63-1d1b-4736-9aba-a87a258b2b11/7a7dfcf0-39e0-4eb7-9f4b-f66d7afbe41f/dd64c4b9-f40c-48f2-9722-a05c0658867e"
 					(reference "JP2")
@@
 			)
 		)
-		(property "Value" "Conn_02x04_Top_Bottom"
+		(property "Value" "Conn_02x04_Top_Bottom_MountingPin"
 			(at 78.994 72.39 0)
 			(effects

Commit message: Free UART7 for alternative BMS usage
Changed lines of the file:
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@@
 		)
 		(property "Value" "120"
-			(at 234.95 45.212 90)
+			(at 234.95 45.72 90)
 			(show_name no)
 			(do_not_autoplace no)
