File: CoverUI-S2.kicad_sch (KiCad schematic)
At the start: 38 parts, among them J2 Conn_01x36_MountingPin

Commit message: Additional Infos
Connections:
- net LED_D renamed LED_BTN_D
- net LED_STR renamed LED_BTN_STR
Changed lines of the file:
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@@
 		)
 	)
-	(label "LED_D"
+	(label "LED_BTN_D"
 		(at 114.3 78.74 0)
 		(effects
@@
 		)
 	)
-	(label "LED_STR"
+	(label "LED_BTN_STR"
 		(at 186.69 104.14 0)
 		(effects
@@
 		)
 	)
-	(label "LED_D"
+	(label "LED_BTN_D"
 		(at 181.61 114.3 0)
 		(effects
@@
 		)
 	)
-	(label "LED_STR"
+	(label "LED_BTN_STR"
 		(at 114.3 81.28 0)
 		(effects

Commit message: v0.2 required changes
Connections:
- net RST: now reaches J2.19 (Pin_19), S2-J?.24 (Pin_24)
- net ID1: now reaches J2.10 (Pin_10), R8.2
Other:
- note added: "LCDisplay: SABO P/N: SAU12991 Molex P/N: 127810002 Date: 13/02/22 LCD: PCBS100058A-2 Counted 240*160 pixel"
- note removed: "LCDisplay: Molex P/N: 127810002 Date: 13/02/22 LCD: PCBS100058A-2"
Changed lines of the file:
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@@
 		(rev "v0.1")
 	)
-	(text "LCDisplay:\nMolex P/N: 127810002\nDate: 13/02/22\n\nLCD: PCBS100058A-2"
+	(text "LCDisplay:\nSABO P/N: SAU12991\nMolex P/N: 127810002\nDate: 13/02/22\n\nLCD: PCBS100058A-2\n\nCounted 240*160 pixel"
 		(exclude_from_sim no)
-		(at 72.644 189.738 0)
+		(at 72.644 186.944 0)
 		(effects
 			(font
@@
 		)
 	)
+	(label "SCK"
+		(at 68.58 147.32 180)
+		(effects
+			(font
+				(size 1.27 1.27)
+			)
+			(justify right bottom)
+		)
+	)
 	(label "LED_BTN_D"
 		(at 114.3 78.74 0)
@@
 		)
 	)
+	(label "VDD"
+		(at 99.06 132.08 0)
+		(effects
+			(font
+				(size 1.27 1.27)
+			)
+			(justify left bottom)
+		)
+	)
+	(label "~{C}D"
+		(at 78.74 148.59 180)
+		(effects
+			(font
+				(size 1.27 1.27)
+			)
+			(justify right bottom)
+		)
+	)
 	(label "~{PL}"
 		(at 240.03 58.42 0)
@@
 	)
 	(label "MB-LM317LM-Pin3_VOut"
-		(at 102.87 132.08 0)
+		(at 118.11 132.08 0)
 		(effects
 			(font
@@
 		)
 	)
+	(label "SDA"
+		(at 48.26 147.32 0)
+		(effects
+			(font
+				(size 1.27 1.27)
+			)
+			(justify left bottom)
+		)
+	)
+	(label "ID1"
+		(at 93.98 154.94 0)
+		(effects
+			(font
+				(size 1.27 1.27)
+			)
+			(justify left bottom)
+		)
+	)
 	(label "BTN_~{CE}"
 		(at 148.59 73.66 180)
@@
 		)
 	)
+	(label "RST"
+		(at 71.12 154.94 0)
+		(effects
+			(font
+				(size 1.27 1.27)
+			)
+			(justify left bottom)
+		)
+	)
