File: AuxPSU.kicad_sch (KiCad schematic)
At the start: 10 parts, among them U4 TPS5430DDA

Commit message: BOM optimization
Other:
- title: OpenMower SABO Mainboard for Series I & II -> OpenMower SABO Carrierboard for Series I & II
Changed lines of the file:
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@@
 	(paper "A3")
 	(title_block
-		(title "OpenMower SABO Mainboard for Series I & II")
-		(date "2025-10-05")
-		(rev "v0.3")
+		(title "OpenMower SABO Carrierboard for Series I & II")
+		(date "2025-10-12")
+		(rev "v0.4")
 		(company "Apeheanger <joerg@ebeling.ws> for OpenMower")
 		(comment 1 "This design is licensed under CC BY-NC 4.0")
