File: AuxPSU.kicad_sch (KiCad schematic)
At the start: 10 parts, among them U4 TPS5430DDA

Commit message: Prepare for next production - Slightly adapt part selection - Add TC2050 holes
Parts:
- C11, C16: JLC C13585 -> (none); LCSC Part # (none) -> C13585
- C12: JLC C1710 -> (none); LCSC Part # (none) -> C1710
- C13: JLC C22387801 -> (none); LCSC Part # (none) -> C22387801
- D16: JLC C22452 -> (none); LCSC Part # (none) -> C22452
- L3: JLC C408489 -> (none); LCSC Part # (none) -> C408489
- R44: JLC C4328 -> (none); LCSC Part # (none) -> C4328
- R45: JLC C17520 -> (none); LCSC Part # (none) -> C17520
- R46: JLC C25744 -> (none); LCSC Part # (none) -> C25744
- U4: JLC C9864 -> (none); LCSC Part # (none) -> C9864
Changed lines of the file:
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@@
-			)
-		)
-		(property "JLC" "C408489"
-			(at 223.52 123.19 0)
-			(effects
-				(font
-					(size 1.27 1.27)
-				)
-				(hide yes)
 			)
 		)
@@
 			)
 		)
-		(property "LCSC" ""
+		(property "LCSC Part #" "C408489"
 			(at 223.52 123.19 90)
 			(effects
@@
 			)
 		)
-		(property "JLC" "C25744"
-			(at 149.86 137.16 0)
-			(effects
-				(font
-					(size 1.27 1.27)
-				)
-				(hide yes)
-			)
-		)
 		(property "Alternative" ""
 			(at 149.86 137.16 90)
@@
 			)
 		)
-		(property "LCSC" ""
+		(property "LCSC Part #" "C25744"
 			(at 149.86 137.16 90)
 			(effects
@@
 			)
 		)
-		(property "JLC" "C4328"
-			(at 237.49 129.54 0)
-			(effects
-				(font
-					(size 1.27 1.27)
-				)
-				(hide yes)
-			)
-		)
 		(property "Alternative" ""
 			(at 237.49 129.54 0)
@@
 			)
 		)
-		(property "LCSC" ""
+		(property "LCSC Part #" "C4328"
 			(at 237.49 129.54 0)
 			(effects
@@
 			)
 		)
-		(property "JLC" "C9864"
-			(at 166.37 128.27 0)
-			(effects
-				(font
-					(size 1.27 1.27)
-				)
-				(hide yes)
-			)
-		)
 		(property "Alternative" ""
 			(at 166.37 128.27 0)
@@
 			)
 		)
-		(property "LCSC" ""
+		(property "LCSC Part #" "C9864"
 			(at 166.37 128.27 0)
 			(effects
@@
 			)
 		)
-		(property "JLC" "C17520"
-			(at 237.49 139.7 0)
-			(effects
-				(font
-					(size 1.27 1.27)
-				)
-				(hide yes)
-			)
-		)
 		(property "Alternative" ""
 			(at 237.49 139.7 0)
@@
 			)
 		)
-		(property "LCSC" ""
+		(property "LCSC Part #" "C17520"
 			(at 237.49 139.7 0)
 			(effects
@@
 			)
 		)
-		(property "JLC" "C13585"
-			(at 125.73 127 0)
-			(effects
-				(font
-					(size 1.27 1.27)
-				)
-				(hide yes)
-			)
-		)
 		(property "Alternative" ""
 			(at 125.73 127 0)
@@
 			)
 		)
-		(property "LCSC" ""
+		(property "LCSC Part #" "C13585"
 			(at 125.73 127 0)
 			(effects
@@
 			)
 		)
-		(property "JLC" "C13585"
-			(at 273.05 127 0)
-			(effects
-				(font
-					(size 1.27 1.27)
-				)
-				(hide yes)
-			)
-		)
 		(property "Alternative" ""
 			(at 273.05 127 0)
@@
 			)
 		)
-		(property "LCSC" ""
+		(property "LCSC Part #" "C13585"
 			(at 273.05 127 0)
 			(effects
@@
 			)
 		)
-		(property "JLC" "C22452"
-			(at 207.01 132.08 90)
-			(effects
-				(font
-					(size 1.27 1.27)
-				)
-				(hide yes)
-			)
-		)
 		(property "Alternative" ""
 			(at 207.01 132.08 90)
@@
 			)
 		)
-		(property "LCSC" ""
+		(property "LCSC Part #" "C22452"
 			(at 207.01 132.08 90)
 			(effects
@@
 			)
 		)
-		(property "JLC" "C22387801"
-			(at 259.08 128.27 0)
-			(effects
-				(font
-					(size 1.27 1.27)
-				)
-				(hide yes)
-			)
-		)
 		(property "FT Rotation Offset" "180"
 			(at 259.08 128.27 0)
@@
 			)
 		)
-		(property "LCSC" ""
+		(property "LCSC Part #" "C22387801"
 			(at 259.08 128.27 0)
 			(effects
@@
 			)
 		)
-		(property "JLC" "C1710"
-			(at 187.96 123.19 0)
-			(effects
-				(font
-					(size 1.27 1.27)
-				)
-				(hide yes)
-			)
-		)
 		(property "Alternative" ""
 			(at 187.96 123.19 90)
@@
 			)
 		)
-		(property "LCSC" ""
+		(property "LCSC Part #" "C1710"
 			(at 187.96 123.19 90)
 			(effects
