File: AuxPSU.kicad_sch (KiCad schematic)
At the start: 10 parts, among them U4 TPS5430DDA

Commit message: Production preparation
Parts:
- C11, C16: LCSC Part # C13585 -> C33546013; MF (none) -> Chinocera; MFPN (none) -> HGC1206R7106K500NSPJ
