File: Amplifier.kicad_sch (KiCad schematic)
At the start: 7 parts, among them U3 MAX98357A

Commit message: Prepare for next production - Slightly adapt part selection - Add TC2050 holes
Parts:
- C10: JLC C307331 -> (none); LCSC Part # (none) -> C307331
- C9: JLC C15008 -> (none); LCSC Part # (none) -> C15008
- R5, R6, R7: JLC C17514 -> (none); LCSC Part # (none) -> C17514
- R8: JLC C17477 -> (none); LCSC Part # (none) -> C17477
- U3: footprint Package_DFN_QFN:TQFN-16-1EP_3x3mm_P0.5mm_EP1.23x1.23mm -> easyeda2kicad:TQFN-16_L3.0-W3.0-P0.50-BL-EP1.5; JLC C910544 -> (none); LCSC Part # (none) -> C910544
Changed lines of the file:
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@@
 			)
 		)
-		(property "Footprint" "Package_DFN_QFN:TQFN-16-1EP_3x3mm_P0.5mm_EP1.23x1.23mm"
+		(property "Footprint" "easyeda2kicad:TQFN-16_L3.0-W3.0-P0.50-BL-EP1.5"
 			(at 151.13 111.76 0)
 			(effects
@@
 			)
 		)
-		(property "JLC" "C910544"
-			(at 152.4 109.22 0)
-			(effects
-				(font
-					(size 1.27 1.27)
-				)
-				(hide yes)
-			)
-		)
 		(property "FT Rotation Offset" "-90"
 			(at 152.4 109.22 0)
@@
 			)
 		)
-		(property "LCSC" ""
+		(property "LCSC Part #" "C910544"
 			(at 152.4 109.22 0)
 			(effects
@@
 			)
 		)
-		(property "JLC" "C17514"
-			(at 104.14 113.03 0)
-			(effects
-				(font
-					(size 1.27 1.27)
-				)
-				(hide yes)
-			)
-		)
 		(property "Alternative" ""
 			(at 104.14 113.03 0)
@@
 			)
 		)
-		(property "LCSC" ""
+		(property "LCSC Part #" "C17514"
 			(at 104.14 113.03 0)
 			(effects
@@
 			)
 		)
-		(property "JLC" "C15008"
-			(at 68.58 71.12 0)
-			(effects
-				(font
-					(size 1.27 1.27)
-				)
-				(hide yes)
-			)
-		)
 		(property "Alternative" ""
 			(at 68.58 71.12 90)
@@
 			)
 		)
-		(property "LCSC" ""
+		(property "LCSC Part #" "C15008"
 			(at 68.58 71.12 90)
 			(effects
@@
 			)
 		)
-		(property "JLC" "C17514"
-			(at 104.14 124.46 0)
-			(effects
-				(font
-					(size 1.27 1.27)
-				)
-				(hide yes)
-			)
-		)
 		(property "Alternative" ""
 			(at 104.14 124.46 0)
@@
 			)
 		)
-		(property "LCSC" ""
+		(property "LCSC Part #" "C17514"
 			(at 104.14 124.46 0)
 			(effects
@@
 			)
 		)
-		(property "JLC" "C17514"
-			(at 120.65 129.54 0)
-			(effects
-				(font
-					(size 1.27 1.27)
-				)
-				(hide yes)
-			)
-		)
 		(property "Alternative" ""
 			(at 120.65 129.54 0)
@@
 			)
 		)
-		(property "LCSC" ""
+		(property "LCSC Part #" "C17514"
 			(at 120.65 129.54 0)
 			(effects
@@
 			)
 		)
-		(property "JLC" "C17477"
-			(at 120.65 140.97 0)
-			(effects
-				(font
-					(size 1.27 1.27)
-				)
-				(hide yes)
-			)
-		)
 		(property "Alternative" ""
 			(at 120.65 140.97 0)
@@
 			)
 		)
-		(property "LCSC" ""
+		(property "LCSC Part #" "C17477"
 			(at 120.65 140.97 0)
 			(effects
@@
 			)
 		)
-		(property "JLC" "C307331"
-			(at 81.28 71.12 0)
-			(effects
-				(font
-					(size 1.27 1.27)
-				)
-				(hide yes)
-			)
-		)
 		(property "Alternative" ""
 			(at 81.28 71.12 0)
@@
 			)
 		)
-		(property "LCSC" ""
+		(property "LCSC Part #" "C307331"
 			(at 81.28 71.12 0)
 			(effects

Commit message: Production state
Parts:
- U3: FT Rotation Offset -90 -> 0
Changed lines of the file:
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@@
 	(title_block
 		(title "OpenMower SABO Carrierboard for Series I & II")
-		(date "2025-10-12")
+		(date "2026-04-04")
 		(rev "v0.4")
 		(company "Apeheanger <joerg@ebeling.ws> for OpenMower")
@@
 			)
 		)
-		(property "FT Rotation Offset" "-90"
+		(property "FT Rotation Offset" "0"
 			(at 152.4 109.22 0)
 			(effects
