File: Charger.kicad_sch (KiCad schematic)
At the start: 58 parts, among them Q6 BSC0702LS, Q7 BSC0702LS, Q8 BSC0702LS, Q9 BSC0702LS, U27 BQ25756RRVR

Commit message: Next proto prep
Parts:
- C80: LCSC Part # C354368 -> C28323
Changed lines of the file:
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@@
 			)
 		)
-		(property "Description" "Unpolarized capacitor"
+		(property "Description" "1uF 50V X7R ±10% 0805 Multilayer Ceramic Capacitors MLCC - SMD/SMT ROHS"
 			(at 100.33 93.98 0)
 			(effects
@@
 			)
 		)
-		(property "LCSC Part #" "C354368"
+		(property "LCSC Part #" "C28323"
 			(at 100.33 93.98 0)
 			(effects

Commit message: Production state
Parts:
- added C22: 4.7uF@50V, Capacitor_SMD:C_1206_3216Metric, symbol Device:C
- added R78, R79: 10R, Resistor_SMD:R_0603_1608Metric, symbol Device:R
- C42, C61: value 100uF@63V -> 220uF@80V; footprint Capacitor_THT:CP_Radial_D8.0mm_P3.50mm -> Capacitor_THT:CP_Radial_D10.0mm_P5.00mm; LCSC Part # C7436417 -> C2937593
- C62, C77: value 100nF -> 100nF@100V; footprint Capacitor_SMD:C_0402_1005Metric -> Capacitor_SMD:C_0805_2012Metric; LCSC Part # C307331 -> C28233
- R33: value 249kR 0.1% -> 249k 0.1%
- R72: value 5.24kR -> 5k1; LCSC Part # (none) -> C23186; now fitted
- R73: value 30.31kR -> 30k; LCSC Part # (none) -> C22984; now fitted
Connections:
- net GND: now also C22.2
- net V_CHARGER: now also C22.1, R78.1; no longer C62.1, C85.2, U27.30 (ACP)
- net at C40.1, C41.1, C61.1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: now also R79.1; no longer C77.2, C85.1, U27.29 (ACN)
- new net: C77.2, C85.1, R79.2, U27.29 (ACN)
- new net: C62.1, C85.2, R78.2, U27.30 (ACP)
Other:
- note added: "103AT-2 (10k thermistor)"
- note added: "R_{AC_SNS} = 5mOhm = 12A * 2/5 = 4.8A I_{Sense_Max}"
- note removed: "R_{AC_SNS} = 5mOhm = 12A * 2/5 = 4.8A I_{Sense_Max} TODO: - Set corresponding regsiter to 0x60?"
- moved on the sheet: C38, C39, C40, C41, C61, C62, C77, C85, R20

Commit message: KiCAD 10.x, Mow-ESC-Fuse, Improve power traces
Parts:
- R78, R79: footprint Resistor_SMD:R_0603_1608Metric -> (none)
