File: xESC.kicad_sch (KiCad schematic)
At the start: 16 parts, among them U18 2.54mm 2x2 socket, U21 2.54mm 2x2 socket, U24 2.54mm 2x2 socket, U30 2.54mm 1x6 socket, U33 2.54mm 1x6 socket, U36 2.54mm 1x9 socket, U39 2.54mm 1x5 socket, U8 xESC2

Commit message: Prepare for next production - Slightly adapt part selection - Add TC2050 holes
Parts:
- C64, C65: JLC C2937593 -> (none); LCSC Part # (none) -> C2937593
- C66, C67: JLC C13585 -> (none); LCSC Part # (none) -> C13585
- U18, U21, U24: footprint xtech:Dummy -> xtech:Dummy_xESC_2x2PH
- U30, U33: footprint xtech:Dummy -> xtech:Dummy_xESC_6PH
- U36: footprint xtech:Dummy -> xtech:Dummy_xESC_9PH
- U39: footprint xtech:Dummy -> xtech:Dummy_xESC_5PH

Commit message: Next proto prep
Parts:
- U18, U21, U24: LCSC Part # C92273 -> C2840016
Changed lines of the file:
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@@
 			)
 		)
-		(property "Description" ""
+		(property "Description" "-40℃~+105℃ 2 2.54mm 2.54mm 250V 2x2P 3A 4P 8.5mm Square Hole Through Hole Top,P=2.54mm Female Headers ROHS"
 			(at 68.58 207.01 0)
 			(effects
@@
 			)
 		)
-		(property "LCSC Part #" "C92273"
+		(property "LCSC Part #" "C2840016"
 			(at 68.58 207.01 0)
 			(effects
@@
 			)
 		)
-		(property "Description" ""
+		(property "Description" "-40℃~+105℃ 2 2.54mm 2.54mm 250V 2x2P 3A 4P 8.5mm Square Hole Through Hole Top,P=2.54mm Female Headers ROHS"
 			(at 68.58 214.63 0)
 			(effects
@@
 			)
 		)
-		(property "LCSC Part #" "C92273"
+		(property "LCSC Part #" "C2840016"
 			(at 68.58 214.63 0)
 			(effects
@@
 			)
 		)
-		(property "Description" ""
+		(property "Description" "-40℃~+105℃ 2 2.54mm 2.54mm 250V 2x2P 3A 4P 8.5mm Square Hole Through Hole Top,P=2.54mm Female Headers ROHS"
 			(at 68.58 222.25 0)
 			(effects
@@
 			)
 		)
-		(property "LCSC Part #" "C92273"
+		(property "LCSC Part #" "C2840016"
 			(at 68.58 222.25 0)
 			(effects
