File: GPS.kicad_sch (KiCad schematic)
At the start: 7 parts, among them Q1 BSS138, U46 2.54mm 2x6 socket

Commit message: BOM optimization
Other:
- title: OpenMower SABO Mainboard for Series I & II -> OpenMower SABO Carrierboard for Series I & II
Changed lines of the file:
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@@
 	(paper "A3")
 	(title_block
-		(title "OpenMower SABO Mainboard for Series I & II")
-		(date "2025-10-05")
-		(rev "v0.3")
+		(title "OpenMower SABO Carrierboard for Series I & II")
+		(date "2025-10-12")
+		(rev "v0.4")
 		(company "Apeheanger <joerg@ebeling.ws> for OpenMower")
 		(comment 1 "This design is licensed under CC BY-NC 4.0")

Commit message: Prepare for next production - Slightly adapt part selection - Add TC2050 holes
Parts:
- Q1: JLC C3040446 -> (none); LCSC Part # (none) -> C3040446
- R24: JLC C17414 -> (none); LCSC Part # (none) -> C17414
- R25: JLC C17471 -> (none); LCSC Part # (none) -> C17471
- R58: JLC C17520 -> (none); LCSC Part # (none) -> C17520
- U46: footprint xtech:Dummy -> xtech:Dummy_GPS_2x6PH
Changed lines of the file:
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@@
-			)
-		)
-		(property "MPN" ""
-			(at 184.15 107.95 0)
-			(effects
-				(font
-					(size 1.27 1.27)
-				)
 			)
 		)
 		(property "Alternative" ""
-			(at 184.15 107.95 0)
-			(effects
-				(font
-					(size 1.27 1.27)
-				)
-				(hide yes)
-			)
-		)
-		(property "LCSC" ""
 			(at 184.15 107.95 0)
 			(effects
@@
 			)
 		)
-		(property "JLC" "C17520"
-			(at 217.17 97.79 0)
-			(effects
-				(font
-					(size 1.27 1.27)
-				)
-				(hide yes)
-			)
-		)
-		(property "MPN" ""
-			(at 217.17 97.79 0)
-			(effects
-				(font
-					(size 1.27 1.27)
-				)
-			)
-		)
 		(property "Alternative" ""
 			(at 217.17 97.79 90)
@@
 			)
 		)
-		(property "LCSC" ""
+		(property "LCSC Part #" "C17520"
 			(at 217.17 97.79 90)
 			(effects
@@
 			)
 		)
-		(property "JLC" "C17414"
-			(at 139.7 115.57 0)
-			(effects
-				(font
-					(size 1.27 1.27)
-				)
-				(hide yes)
-			)
-		)
-		(property "MPN" ""
-			(at 139.7 115.57 0)
-			(effects
-				(font
-					(size 1.27 1.27)
-				)
-			)
-		)
 		(property "Alternative" ""
 			(at 139.7 115.57 0)
@@
 			)
 		)
-		(property "LCSC" ""
+		(property "LCSC Part #" "C17414"
 			(at 139.7 115.57 0)
 			(effects
@@
 			)
 		)
-		(property "MPN" ""
-			(at 124.46 60.96 0)
-			(effects
-				(font
-					(size 1.27 1.27)
-				)
-			)
-		)
 		(property "Alternative" ""
-			(at 124.46 60.96 0)
-			(effects
-				(font
-					(size 1.27 1.27)
-				)
-				(hide yes)
-			)
-		)
-		(property "LCSC" ""
 			(at 124.46 60.96 0)
 			(effects
@@
 			)
 		)
-		(property "JLC" "C17471"
-			(at 147.32 107.95 0)
-			(effects
-				(font
-					(size 1.27 1.27)
-				)
-				(hide yes)
-			)
-		)
-		(property "MPN" ""
-			(at 147.32 107.95 0)
-			(effects
-				(font
-					(size 1.27 1.27)
-				)
-			)
-		)
 		(property "Alternative" ""
 			(at 147.32 107.95 90)
@@
 			)
 		)
-		(property "LCSC" ""
+		(property "LCSC Part #" "C17471"
 			(at 147.32 107.95 90)
 			(effects
@@
 			)
 		)
-		(property "Footprint" "xtech:Dummy"
+		(property "Footprint" "xtech:Dummy_GPS_2x6PH"
 			(at 354.33 31.75 0)
 			(effects
@@
 			)
 		)
-		(property "JLC" ""
-			(at 354.33 31.75 0)
-			(effects
-				(font
-					(size 1.27 1.27)
-				)
-				(hide yes)
-			)
-		)
-		(property "MPN" ""
-			(at 354.33 31.75 0)
-			(effects
-				(font
-					(size 1.27 1.27)
-				)
-			)
-		)
 		(property "LCSC Part #" "C718230"
 			(at 354.33 31.75 0)
@@
 		)
 		(property "Alternative" ""
-			(at 354.33 31.75 0)
-			(effects
-				(font
-					(size 1.27 1.27)
-				)
-				(hide yes)
-			)
-		)
-		(property "LCSC" ""
 			(at 354.33 31.75 0)
 			(effects
@@
 			)
 		)
-		(property "JLC" "C3040446"
-			(at 160.02 107.95 0)
-			(effects
-				(font
-					(size 1.27 1.27)
-				)
-				(hide yes)
-			)
-		)
-		(property "MPN" ""
-			(at 160.02 107.95 0)
-			(effects
-				(font
-					(size 1.27 1.27)
-				)
-			)
-		)
 		(property "Alternative" ""
 			(at 160.02 107.95 0)
@@
 			)
 		)
-		(property "LCSC" ""
+		(property "LCSC Part #" "C3040446"
 			(at 160.02 107.95 0)
 			(effects

Commit message: Next proto prep
Parts:
- Q1: value BSS138 -> AO3400A; LCSC Part # C3040446 -> C20917
Changed lines of the file:
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@@
 			)
 		)
-		(property "Value" "BSS138"
+		(property "Value" "AO3400A"
 			(at 164.846 109.474 0)
 			(effects
@@
 			)
 		)
-		(property "Description" "50V Vds, 0.22A Id, N-Channel MOSFET, SOT-23"
+		(property "Description" "-55℃~+150℃ 1 N-channel 1.45V 1.4W 30V 48mΩ@2.5V 5.7A 50pF 630pF 75pF 7nC@10V N-Channel SOT-23-3L MOSFETs ROHS"
 			(at 160.02 107.95 0)
 			(effects
@@
 			)
 		)
-		(property "LCSC Part #" "C3040446"
+		(property "LCSC Part #" "C20917"
 			(at 160.02 107.95 0)
 			(effects

Commit message: KiCAD 10.x, Mow-ESC-Fuse, Improve power traces
Parts:
- U13: value ~ -> (none)

Commit message: Free UART7 for alternative BMS usage
Parts:
- R58: value 2.2k -> 1k; footprint Resistor_SMD:R_0805_2012Metric -> Resistor_SMD:R_0402_1005Metric; LCSC Part # C17520 -> C11702
Changed lines of the file:
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@@
 			)
 		)
-		(property "Value" "2.2k"
+		(property "Value" "1k"
 			(at 217.424 103.124 90)
 			(show_name no)
@@
 			)
 		)
-		(property "Footprint" "Resistor_SMD:R_0805_2012Metric"
+		(property "Footprint" "Resistor_SMD:R_0402_1005Metric"
 			(at 217.17 99.568 90)
 			(hide yes)
@@
 			)
 		)
-		(property "Description" "Resistor"
+		(property "Description" "-55℃~+155℃ 1kΩ 50V 62.5mW Thick Film Resistor ±1% ±100ppm/℃ 0402 Chip Resistor - Surface Mount ROHS"
 			(at 217.17 97.79 0)
 			(hide yes)
@@
 			)
 		)
-		(property "LCSC Part #" "C17520"
+		(property "LCSC Part #" "C11702"
 			(at 217.17 97.79 90)
 			(hide yes)
