File: Core.kicad_sch (KiCad schematic)
At the start: 1 part, among them J26 xcore

Commit message: Prepare for next production - Slightly adapt part selection - Add TC2050 holes
Parts:
- J26: value xcore -> SODIMM 204P; JLC C306045 -> (none); JLC-ALT C225721 -> C306045; LCSC Part # (none) -> C225721
Changed lines of the file:
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@@
 			)
 		)
-		(property "Value" "xcore"
+		(property "Value" "SODIMM 204P"
 			(at 204.47 137.7949 0)
 			(effects
@@
 			)
 		)
-		(property "JLC" "C306045"
-			(at 193.04 139.7 0)
-			(effects
-				(font
-					(size 1.27 1.27)
-				)
-				(hide yes)
-			)
-		)
 		(property "Alt" "TE Connectivity 2-2013289-1"
 			(at 193.04 139.7 0)
@@
 			)
 		)
-		(property "JLC-ALT" "C225721"
+		(property "JLC-ALT" "C306045"
 			(at 193.04 139.7 0)
 			(effects
@@
 			)
 		)
-		(property "MPN" ""
-			(at 193.04 139.7 0)
-			(effects
-				(font
-					(size 1.27 1.27)
-				)
-			)
-		)
 		(property "Alternative" ""
 			(at 193.04 139.7 0)
@@
 			)
 		)
-		(property "LCSC" ""
+		(property "LCSC Part #" "C225721"
 			(at 193.04 139.7 0)
 			(effects
@@
 			)
 		)
-		(property "Value" "xcore"
+		(property "Value" "SODIMM 204P"
 			(at 101.6 62.8649 0)
 			(effects
@@
 			)
 		)
-		(property "JLC" "C306045"
-			(at 88.9 60.96 0)
-			(effects
-				(font
-					(size 1.27 1.27)
-				)
-				(hide yes)
-			)
-		)
 		(property "Alt" "TE Connectivity 2-2013289-1"
 			(at 88.9 60.96 0)
@@
 			)
 		)
-		(property "JLC-ALT" "C225721"
+		(property "JLC-ALT" "C306045"
 			(at 88.9 60.96 0)
 			(effects
@@
 			)
 		)
-		(property "MPN" ""
-			(at 88.9 60.96 0)
-			(effects
-				(font
-					(size 1.27 1.27)
-				)
-			)
-		)
 		(property "Alternative" ""
 			(at 88.9 60.96 0)
@@
 			)
 		)
-		(property "LCSC" ""
+		(property "LCSC Part #" "C225721"
 			(at 88.9 60.96 0)
 			(effects
@@
 			)
 		)
-		(property "Value" "xcore"
+		(property "Value" "SODIMM 204P"
 			(at 276.86 164.4649 0)
 			(effects
@@
 			)
 		)
-		(property "JLC" "C306045"
-			(at 262.89 152.4 0)
-			(effects
-				(font
-					(size 1.27 1.27)
-				)
-				(hide yes)
-			)
-		)
 		(property "Alt" "TE Connectivity 2-2013289-1"
 			(at 262.89 152.4 0)
@@
 			)
 		)
-		(property "JLC-ALT" "C225721"
+		(property "JLC-ALT" "C306045"
 			(at 262.89 152.4 0)
 			(effects
@@
 			)
 		)
-		(property "MPN" ""
-			(at 262.89 152.4 0)
-			(effects
-				(font
-					(size 1.27 1.27)
-				)
-			)
-		)
 		(property "Alternative" ""
 			(at 262.89 152.4 0)
@@
 			)
 		)
-		(property "LCSC" ""
+		(property "LCSC Part #" "C225721"
 			(at 262.89 152.4 0)
 			(effects
@@
 			)
 		)
-		(property "Value" "xcore"
+		(property "Value" "SODIMM 204P"
 			(at 276.86 90.1699 0)
 			(effects
@@
 			)
 		)
-		(property "JLC" "C306045"
-			(at 264.16 91.44 0)
-			(effects
-				(font
-					(size 1.27 1.27)
-				)
-				(hide yes)
-			)
-		)
 		(property "Alt" "TE Connectivity 2-2013289-1"
 			(at 264.16 91.44 0)
@@
 			)
 		)
-		(property "JLC-ALT" "C225721"
+		(property "JLC-ALT" "C306045"
 			(at 264.16 91.44 0)
 			(effects
@@
 			)
 		)
-		(property "MPN" ""
-			(at 264.16 91.44 0)
-			(effects
-				(font
-					(size 1.27 1.27)
-				)
-			)
-		)
 		(property "Alternative" ""
 			(at 264.16 91.44 0)
@@
 			)
 		)
-		(property "LCSC" ""
+		(property "LCSC Part #" "C225721"
 			(at 264.16 91.44 0)
 			(effects
@@
 			)
 		)
-		(property "Value" "xcore"
+		(property "Value" "SODIMM 204P"
 			(at 87.63 115.57 0)
 			(effects
@@
 			)
 		)
-		(property "JLC" "C306045"
-			(at 87.63 152.4 0)
-			(effects
-				(font
-					(size 1.27 1.27)
-				)
-				(hide yes)
-			)
-		)
 		(property "Alt" "TE Connectivity 2-2013289-1"
 			(at 87.63 152.4 0)
@@
 			)
 		)
-		(property "JLC-ALT" "C225721"
+		(property "JLC-ALT" "C306045"
 			(at 87.63 152.4 0)
 			(effects
@@
 			)
 		)
-		(property "MPN" ""
-			(at 87.63 152.4 0)
-			(effects
-				(font
-					(size 1.27 1.27)
-				)
-			)
-		)
 		(property "Alternative" ""
 			(at 87.63 152.4 0)
@@
 			)
 		)
-		(property "LCSC" ""
+		(property "LCSC Part #" "C225721"
 			(at 87.63 152.4 0)
 			(effects
